Commit message: lego built version 1

File: locosim/robot_descriptions/ur_description/urdf/inc/tavolo.xacro (robot description, xacro)
@@ -47,5 +47,5 @@
     </collision>
     <!-- Back collision -->
-    <collision name="back_collision">
+    <!-- <collision name="back_collision">
       <origin xyz="0.5 -0.02 1.35" rpy="1.57 0 0"/>
       <geometry>
@@ -60,5 +60,5 @@
         </friction>
       </surface>
-    </collision>
+    </collision> -->
   </link>
 </robot>
